File: hardware/logicboard/mb-001.brd (EAGLE design)
At the start: 91 x 57 mm, 11 parts, among them J1 DIN5, J2 DIN5, J3 DIN5, J4 AUDIO_JACK_3.5MM_KIT, J5 AUDIO_JACK_3.5MM_KIT, J6 AUDIO_JACK_3.5MM_KIT

Commit message: Symbol name.
Parts:
- renumbered J4 to JJ1, J5 to JJ2, J6 to JJ3
Changed lines of the file:
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@@
 <attribute name="VALUE" x="27.27" y="53.063" size="0.6096" layer="27" font="vector" ratio="20" rot="R180"/>
 </element>
-<element name="J4" library="SparkFun-Connectors" library_urn="urn:adsk.eagle:library:513" package="AUDIO-JACK-KIT" package3d_urn="urn:adsk.eagle:package:38014/1" value="AUDIO_JACK_3.5MM_KIT" x="65" y="6.5" smashed="yes" rot="R90">
+<element name="JJ1" library="SparkFun-Connectors" library_urn="urn:adsk.eagle:library:513" package="AUDIO-JACK-KIT" package3d_urn="urn:adsk.eagle:package:38014/1" value="AUDIO_JACK_3.5MM_KIT" x="65" y="6.5" smashed="yes" rot="R90">
 <attribute name="NAME" x="65" y="14.5" size="1" layer="25" ratio="20" align="bottom-center"/>
 <attribute name="PROD_ID" value="CONN-08774" x="65" y="6.5" size="1.778" layer="27" rot="R90" display="off"/>
@@
 <attribute name="VALUE" x="67.667" y="5.23" size="0.6096" layer="27" font="vector" ratio="20" rot="R90"/>
 </element>
-<element name="J5" library="SparkFun-Connectors" library_urn="urn:adsk.eagle:library:513" package="AUDIO-JACK-KIT" package3d_urn="urn:adsk.eagle:package:38014/1" value="AUDIO_JACK_3.5MM_KIT" x="45.5" y="6.5" smashed="yes" rot="R90">
+<element name="JJ2" library="SparkFun-Connectors" library_urn="urn:adsk.eagle:library:513" package="AUDIO-JACK-KIT" package3d_urn="urn:adsk.eagle:package:38014/1" value="AUDIO_JACK_3.5MM_KIT" x="45.5" y="6.5" smashed="yes" rot="R90">
 <attribute name="NAME" x="45.5" y="14.5" size="1" layer="25" ratio="20" align="bottom-center"/>
 <attribute name="PROD_ID" value="CONN-08774" x="45.5" y="6.5" size="1.778" layer="27" rot="R90" display="off"/>
@@
 <attribute name="VALUE" x="48.167" y="5.23" size="0.6096" layer="27" font="vector" ratio="20" rot="R90"/>
 </element>
-<element name="J6" library="SparkFun-Connectors" library_urn="urn:adsk.eagle:library:513" package="AUDIO-JACK-KIT" package3d_urn="urn:adsk.eagle:package:38014/1" value="AUDIO_JACK_3.5MM_KIT" x="26" y="6.5" smashed="yes" rot="R90">
+<element name="JJ3" library="SparkFun-Connectors" library_urn="urn:adsk.eagle:library:513" package="AUDIO-JACK-KIT" package3d_urn="urn:adsk.eagle:package:38014/1" value="AUDIO_JACK_3.5MM_KIT" x="26" y="6.5" smashed="yes" rot="R90">
 <attribute name="NAME" x="26" y="14.5" size="1" layer="25" ratio="20" align="bottom-center"/>
 <attribute name="PROD_ID" value="CONN-08774" x="26" y="6.5" size="1.778" layer="27" rot="R90" display="off"/>
@@
 <signal name="M1GND" class="2">
 <contactref element="J1" pad="2"/>
-<contactref element="J4" pad="SLEEVE"/>
+<contactref element="JJ1" pad="SLEEVE"/>
 <wire x1="65.0748" y1="10.1346" x2="65.0748" y2="6.5532" width="0.3048" layer="16"/>
 <wire x1="66.0654" y1="11.1252" x2="65.0748" y2="10.1346" width="0.3048" layer="16"/>
@@
 <signal name="M3GND" class="2">
 <contactref element="J3" pad="2"/>
-<contactref element="J6" pad="SLEEVE"/>
+<contactref element="JJ3" pad="SLEEVE"/>
 <wire x1="26.0604" y1="10.1346" x2="26.0604" y2="6.5532" width="0.3048" layer="16"/>
 <wire x1="27.051" y1="11.1252" x2="26.0604" y2="10.1346" width="0.3048" layer="16"/>
@@
 <signal name="M2GND" class="2">
 <contactref element="J2" pad="2"/>
-<contactref element="J5" pad="SLEEVE"/>
+<contactref element="JJ2" pad="SLEEVE"/>
 <wire x1="45.5676" y1="10.1346" x2="45.5676" y2="6.5532" width="0.3048" layer="16"/>
 <wire x1="46.5582" y1="11.1252" x2="45.5676" y2="10.1346" width="0.3048" layer="16"/>
@@
 <signal name="M1TIP">
 <contactref element="S1" pad="3"/>
-<contactref element="J4" pad="TIP"/>
+<contactref element="JJ1" pad="TIP"/>
 <contactref element="S1" pad="4"/>
 <wire x1="66.294" y1="17.7546" x2="67.5132" y2="17.7546" width="0.1524" layer="16"/>
@@
 </signal>
 <signal name="M1RNG">
-<contactref element="J4" pad="RING"/>
+<contactref element="JJ1" pad="RING"/>
 <contactref element="S1" pad="6"/>
 <contactref element="S1" pad="1"/>
@@
 <signal name="M2TIP">
 <contactref element="S2" pad="3"/>
-<contactref element="J5" pad="TIP"/>
+<contactref element="JJ2" pad="TIP"/>
 <contactref element="S2" pad="4"/>
 <wire x1="46.7868" y1="17.7546" x2="48.006" y2="17.7546" width="0.1524" layer="16"/>
@@
 <signal name="M2RNG">
 <contactref element="S2" pad="1"/>
-<contactref element="J5" pad="RING"/>
+<contactref element="JJ2" pad="RING"/>
 <contactref element="S2" pad="6"/>
 <wire x1="44.196" y1="17.7546" x2="42.9768" y2="17.7546" width="0.1524" layer="1"/>
@@
 <signal name="M3TIP">
 <contactref element="S3" pad="3"/>
-<contactref element="J6" pad="TIP"/>
+<contactref element="JJ3" pad="TIP"/>
 <contactref element="S3" pad="4"/>
 <wire x1="27.2796" y1="17.7546" x2="28.4988" y2="17.7546" width="0.1524" layer="16"/>
@@
 <contactref element="S3" pad="1"/>
 <contactref element="S3" pad="6"/>
-<contactref element="J6" pad="RING"/>
+<contactref element="JJ3" pad="RING"/>
 <wire x1="24.765" y1="17.7546" x2="23.4696" y2="17.7546" width="0.1524" layer="1"/>
 <wire x1="27.2796" y1="20.2692" x2="24.765" y2="17.7546" width="0.1524" layer="1"/>

Commit message: Symbol name.
Parts:
- renumbered J1 to J7, J2 to J8, J3 to J9, JJ1 to JJ7, JJ2 to JJ8, JJ3 to JJ9
Changed lines of the file:
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@@
 <element name="LOGO1" library="SparkFun-Aesthetics" package="OSHW-LOGO-S_COPPER" value="OSHW-LOGOS-COPPER" x="45.5" y="35.5" smashed="yes"/>
 <element name="U$1" library="pineapple" package="PINEAPPLE450" value="PINEAPPLE450" x="45.5" y="28.5" smashed="yes"/>
-<element name="J1" library="SparkFun-Connectors" library_urn="urn:adsk.eagle:library:513" package="DIN5-RA-PTH" package3d_urn="urn:adsk.eagle:package:38294/1" value="DIN5" x="65" y="57" smashed="yes" rot="R180">
+<element name="J7" library="SparkFun-Connectors" library_urn="urn:adsk.eagle:library:513" package="DIN5-RA-PTH" package3d_urn="urn:adsk.eagle:package:38294/1" value="DIN5" x="65" y="57" smashed="yes" rot="R180">
 <attribute name="NAME" x="69" y="38" size="1" layer="25" ratio="20" align="center"/>
 <attribute name="PROD_ID" value="CONN-09481" x="65" y="57" size="1.778" layer="27" rot="R180" display="off"/>
 <attribute name="VALUE" x="66.27" y="53.063" size="0.6096" layer="27" font="vector" ratio="20" rot="R180"/>
 </element>
-<element name="J2" library="SparkFun-Connectors" library_urn="urn:adsk.eagle:library:513" package="DIN5-RA-PTH" package3d_urn="urn:adsk.eagle:package:38294/1" value="DIN5" x="45.5" y="57" smashed="yes" rot="R180">
+<element name="J8" library="SparkFun-Connectors" library_urn="urn:adsk.eagle:library:513" package="DIN5-RA-PTH" package3d_urn="urn:adsk.eagle:package:38294/1" value="DIN5" x="45.5" y="57" smashed="yes" rot="R180">
 <attribute name="NAME" x="49.5" y="38" size="1" layer="25" ratio="20" rot="R180" align="center"/>
 <attribute name="PROD_ID" value="CONN-09481" x="45.5" y="57" size="1.778" layer="27" rot="R180" display="off"/>
 <attribute name="VALUE" x="46.77" y="53.063" size="0.6096" layer="27" font="vector" ratio="20" rot="R180"/>
 </element>
-<element name="J3" library="SparkFun-Connectors" library_urn="urn:adsk.eagle:library:513" package="DIN5-RA-PTH" package3d_urn="urn:adsk.eagle:package:38294/1" value="DIN5" x="26" y="57" smashed="yes" rot="R180">
+<element name="J9" library="SparkFun-Connectors" library_urn="urn:adsk.eagle:library:513" package="DIN5-RA-PTH" package3d_urn="urn:adsk.eagle:package:38294/1" value="DIN5" x="26" y="57" smashed="yes" rot="R180">
 <attribute name="NAME" x="30" y="38" size="1" layer="25" ratio="20" align="center"/>
 <attribute name="PROD_ID" value="CONN-09481" x="26" y="57" size="1.778" layer="27" rot="R180" display="off"/>
 <attribute name="VALUE" x="27.27" y="53.063" size="0.6096" layer="27" font="vector" ratio="20" rot="R180"/>
 </element>
-<element name="JJ1" library="SparkFun-Connectors" library_urn="urn:adsk.eagle:library:513" package="AUDIO-JACK-KIT" package3d_urn="urn:adsk.eagle:package:38014/1" value="AUDIO_JACK_3.5MM_KIT" x="65" y="6.5" smashed="yes" rot="R90">
+<element name="JJ7" library="SparkFun-Connectors" library_urn="urn:adsk.eagle:library:513" package="AUDIO-JACK-KIT" package3d_urn="urn:adsk.eagle:package:38014/1" value="AUDIO_JACK_3.5MM_KIT" x="65" y="6.5" smashed="yes" rot="R90">
 <attribute name="NAME" x="65" y="14.5" size="1" layer="25" ratio="20" align="bottom-center"/>
 <attribute name="PROD_ID" value="CONN-08774" x="65" y="6.5" size="1.778" layer="27" rot="R90" display="off"/>
@@
 <attribute name="VALUE" x="67.667" y="5.23" size="0.6096" layer="27" font="vector" ratio="20" rot="R90"/>
 </element>
-<element name="JJ2" library="SparkFun-Connectors" library_urn="urn:adsk.eagle:library:513" package="AUDIO-JACK-KIT" package3d_urn="urn:adsk.eagle:package:38014/1" value="AUDIO_JACK_3.5MM_KIT" x="45.5" y="6.5" smashed="yes" rot="R90">
+<element name="JJ8" library="SparkFun-Connectors" library_urn="urn:adsk.eagle:library:513" package="AUDIO-JACK-KIT" package3d_urn="urn:adsk.eagle:package:38014/1" value="AUDIO_JACK_3.5MM_KIT" x="45.5" y="6.5" smashed="yes" rot="R90">
 <attribute name="NAME" x="45.5" y="14.5" size="1" layer="25" ratio="20" align="bottom-center"/>
 <attribute name="PROD_ID" value="CONN-08774" x="45.5" y="6.5" size="1.778" layer="27" rot="R90" display="off"/>
@@
 <attribute name="VALUE" x="48.167" y="5.23" size="0.6096" layer="27" font="vector" ratio="20" rot="R90"/>
 </element>
-<element name="JJ3" library="SparkFun-Connectors" library_urn="urn:adsk.eagle:library:513" package="AUDIO-JACK-KIT" package3d_urn="urn:adsk.eagle:package:38014/1" value="AUDIO_JACK_3.5MM_KIT" x="26" y="6.5" smashed="yes" rot="R90">
+<element name="JJ9" library="SparkFun-Connectors" library_urn="urn:adsk.eagle:library:513" package="AUDIO-JACK-KIT" package3d_urn="urn:adsk.eagle:package:38014/1" value="AUDIO_JACK_3.5MM_KIT" x="26" y="6.5" smashed="yes" rot="R90">
 <attribute name="NAME" x="26" y="14.5" size="1" layer="25" ratio="20" align="bottom-center"/>
 <attribute name="PROD_ID" value="CONN-08774" x="26" y="6.5" size="1.778" layer="27" rot="R90" display="off"/>
@@
 <signals>
 <signal name="M1RTN">
-<contactref element="J1" pad="5"/>
+<contactref element="J7" pad="5"/>
 <contactref element="S1" pad="2"/>
 <wire x1="66.294" y1="17.7546" x2="65.0748" y2="17.7546" width="0.1524" layer="1"/>
@@
 </signal>
 <signal name="M3RTN">
-<contactref element="J3" pad="5"/>
+<contactref element="J9" pad="5"/>
 <contactref element="S3" pad="2"/>
 <wire x1="27.2796" y1="17.7546" x2="26.0604" y2="17.7546" width="0.1524" layer="1"/>
@@
 </signal>
 <signal name="M2RTN">
-<contactref element="J2" pad="5"/>
+<contactref element="J8" pad="5"/>
 <contactref element="S2" pad="2"/>
 <wire x1="46.7868" y1="17.7546" x2="45.5676" y2="17.7546" width="0.1524" layer="1"/>
@@
 </signal>
 <signal name="M1GND" class="2">
-<contactref element="J1" pad="2"/>
-<contactref element="JJ1" pad="SLEEVE"/>
+<contactref element="J7" pad="2"/>
+<contactref element="JJ7" pad="SLEEVE"/>
 <wire x1="65.0748" y1="10.1346" x2="65.0748" y2="6.5532" width="0.3048" layer="16"/>
 <wire x1="66.0654" y1="11.1252" x2="65.0748" y2="10.1346" width="0.3048" layer="16"/>
@@
 </signal>
 <signal name="M3GND" class="2">
-<contactref element="J3" pad="2"/>
-<contactref element="JJ3" pad="SLEEVE"/>
+<contactref element="J9" pad="2"/>
+<contactref element="JJ9" pad="SLEEVE"/>
 <wire x1="26.0604" y1="10.1346" x2="26.0604" y2="6.5532" width="0.3048" layer="16"/>
 <wire x1="27.051" y1="11.1252" x2="26.0604" y2="10.1346" width="0.3048" layer="16"/>
@@
 </signal>
 <signal name="M2GND" class="2">
-<contactref element="J2" pad="2"/>
-<contactref element="JJ2" pad="SLEEVE"/>
+<contactref element="J8" pad="2"/>
+<contactref element="JJ8" pad="SLEEVE"/>
 <wire x1="45.5676" y1="10.1346" x2="45.5676" y2="6.5532" width="0.3048" layer="16"/>
 <wire x1="46.5582" y1="11.1252" x2="45.5676" y2="10.1346" width="0.3048" layer="16"/>
@@
 </signal>
 <signal name="M1SND">
-<contactref element="J1" pad="4"/>
+<contactref element="J7" pad="4"/>
 <contactref element="S1" pad="5"/>
 <wire x1="64.9986" y1="37.0332" x2="64.9986" y2="20.3454" width="0.1524" layer="1"/>
@@
 <signal name="M1TIP">
 <contactref element="S1" pad="3"/>
-<contactref element="JJ1" pad="TIP"/>
+<contactref element="JJ7" pad="TIP"/>
 <contactref element="S1" pad="4"/>
 <wire x1="66.294" y1="17.7546" x2="67.5132" y2="17.7546" width="0.1524" layer="16"/>
@@
 </signal>
 <signal name="M1RNG">
-<contactref element="JJ1" pad="RING"/>
+<contactref element="JJ7" pad="RING"/>
 <contactref element="S1" pad="6"/>
 <contactref element="S1" pad="1"/>
@@
 </signal>
 <signal name="M2SND">
-<contactref element="J2" pad="4"/>
+<contactref element="J8" pad="4"/>
 <contactref element="S2" pad="5"/>
 <wire x1="45.4914" y1="37.0332" x2="45.4914" y2="20.3454" width="0.1524" layer="16"/>
@@
 <signal name="M2TIP">
 <contactref element="S2" pad="3"/>
-<contactref element="JJ2" pad="TIP"/>
+<contactref element="JJ8" pad="TIP"/>
 <contactref element="S2" pad="4"/>
 <wire x1="46.7868" y1="17.7546" x2="48.006" y2="17.7546" width="0.1524" layer="16"/>
@@
 <signal name="M2RNG">
 <contactref element="S2" pad="1"/>
-<contactref element="JJ2" pad="RING"/>
+<contactref element="JJ8" pad="RING"/>
 <contactref element="S2" pad="6"/>
 <wire x1="44.196" y1="17.7546" x2="42.9768" y2="17.7546" width="0.1524" layer="1"/>
@@
 </signal>
 <signal name="M3SND">
-<contactref element="J3" pad="4"/>
+<contactref element="J9" pad="4"/>
 <contactref element="S3" pad="5"/>
 <wire x1="25.9842" y1="37.0332" x2="25.9842" y2="20.3454" width="0.1524" layer="1"/>
@@
 <signal name="M3TIP">
 <contactref element="S3" pad="3"/>
-<contactref element="JJ3" pad="TIP"/>
+<contactref element="JJ9" pad="TIP"/>
 <contactref element="S3" pad="4"/>
 <wire x1="27.2796" y1="17.7546" x2="28.4988" y2="17.7546" width="0.1524" layer="16"/>
@@
 <contactref element="S3" pad="1"/>
 <contactref element="S3" pad="6"/>
-<contactref element="JJ3" pad="RING"/>
+<contactref element="JJ9" pad="RING"/>
 <wire x1="24.765" y1="17.7546" x2="23.4696" y2="17.7546" width="0.1524" layer="1"/>
 <wire x1="27.2796" y1="20.2692" x2="24.765" y2="17.7546" width="0.1524" layer="1"/>
